Commit message: add slam hector and cartographer

File: ancubekit_description/urdf/aunchan.xacro (robot description, xacro)
@@ -10,5 +10,5 @@
     <link name="base_link"/>
     <joint name="laser_fixed" type="fixed">
-        <origin xyz="0.01 0 0.19" rpy="0 0 0"/>
+        <origin xyz="-0.01 0 0.19" rpy="0 0 0"/>
         <parent link="base_link"/>
         <child link="laser_link"/>
@@ -16,5 +16,5 @@
     <link name="laser_link"/>
     <joint name="imu_fixed" type="fixed">
-        <origin xyz="0.02 -0.015 0.1" rpy="0 0 0"/>
+        <origin xyz="-0.02 0.015 0.1" rpy="0 0 0"/>
         <parent link="base_link"/>
         <child link="imu_link"/>
